Commit message: some measures fixed

File: src/description_atwork/urdf/arm.xacro (robot description, xacro)
@@ -66,5 +66,5 @@
                 <box size="0.06 0.05 0.1" />
             </geometry>
-            <origin xyz="0 0 0.055" rpy="0 0 0" />
+            <origin xyz="0 0 -0.005" rpy="0 0 0" />
             <material name="grey" />
         </visual>
@@ -73,5 +73,5 @@
                 <box size="0.06 0.05 0.1" />
             </geometry>
-            <origin xyz="0 0 0.055" rpy="0 0 0" />
+            <origin xyz="0 0 -0.005" rpy="0 0 0" />
         </collision>
     </link>
@@ -117,5 +117,5 @@
         <parent link="link_3" />
         <child link="link_4" />
-        <origin xyz="-0.025 0 0.25" rpy="0 0 0" />
+        <origin xyz="-0.025 0 0.295" rpy="0 0 0" />
         <axis xyz="1 0 0" />
         <limit effort="1000.0" velocity="1.0" lower="-1.57" upper="1.57" />
@@ -124,5 +124,5 @@
         <parent link="link_4" />
         <child link="link_5" />
-        <origin xyz="0 0 0.1" rpy="0 0 0" />
+        <origin xyz="0 0 0.045" rpy="0 0 0" />
         <axis xyz="0 0 1" />
         <limit effort="1000.0" velocity="1.0" lower="-3.14" upper="3.14" />
