Commit message: matched with episode 31

File: src/description_atwork/urdf/my_robot.urdf.xacro (robot description, xacro)
@@ -4,4 +4,5 @@
     <xacro:include filename="arm.xacro" />
     <xacro:include filename="gripper.xacro" />
+    <xacro:include filename="my_robot.ros2_control.xacro" />
     <joint name="gripper_base_joint" type="fixed">
         <parent link="tool_link" />

File: src/moveit_config_atwork/config/my_robot.ros2_control.xacro (robot description, xacro)
@@ -38,8 +38,8 @@
                 </state_interface>
             </joint>
-            <joint name="joint6">
+            <joint name="gripper_left_finger_joint">
                 <command_interface name="position"/>
                 <state_interface name="position">
-                  <param name="initial_value">${initial_positions['joint6']}</param>
+                  <param name="initial_value">${initial_positions['gripper_left_finger_joint']}</param>
                 </state_interface>
             </joint>

File: src/moveit_config_atwork/config/my_robot.urdf.xacro (robot description, xacro)
@@ -3,5 +3,5 @@
     <xacro:arg name="initial_positions_file" default="initial_positions.yaml" />
     <!-- Import my_robot urdf file -->
-    <xacro:include filename="$(find description)/urdf/my_robot.urdf.xacro" />
+    <xacro:include filename="$(find description_atwork)/urdf/my_robot.urdf.xacro" />
     <!-- Import control_xacro -->
     <xacro:include filename="my_robot.ros2_control.xacro" />
